Commit message: v0.0.11 重写了仿真

File: software/fly_ROS2_sim/src/fly_simulation/urdf/map.xacro (robot description, xacro)
@@ -4,149 +4,20 @@
     <color rgba="0.3 0.3 0.3 1"/>
   </material>
-  <material name="obstacle_color">
-    <color rgba="0.8 0.2 0.2 1"/>
-  </material>
   <link name="ground">
     <visual>
-      <origin xyz="0 0 -0.01" rpy="0 0 0"/>
       <geometry>
-        <box size="50 50 0.02"/>
+        <box size="100 100 0.01"/>
       </geometry>
       <material name="ground_color"/>
     </visual>
     <collision>
-      <origin xyz="0 0 -0.01" rpy="0 0 0"/>
       <geometry>
-        <box size="50 50 0.02"/>
+        <box size="100 100 0.01"/>
       </geometry>
     </collision>
   </link>
-  <link name="obstacle_1">
-    <visual>
-      <origin xyz="0 0 0" rpy="0 0 0"/>
-      <geometry>
-        <box size="2 2 4"/>
-      </geometry>
-      <material name="obstacle_color"/>
-    </visual>
-    <collision>
-      <geometry>
-        <box size="2 2 4"/>
-      </geometry>
-    </collision>
-  </link>
-  <joint name="obstacle_1_joint" type="fixed">
-    <parent link="ground"/>
-    <child link="obstacle_1"/>
-    <origin xyz="10 10 2" rpy="0 0 0"/>
-  </joint>
-  <link name="obstacle_2">
-    <visual>
-      <origin xyz="0 0 0" rpy="0 0 0"/>
-      <geometry>
-        <box size="3 3 3"/>
-      </geometry>
-      <material name="obstacle_color"/>
-    </visual>
-    <collision>
-      <geometry>
-        <box size="3 3 3"/>
-      </geometry>
-    </collision>
-  </link>
-  <joint name="obstacle_2_joint" type="fixed">
-    <parent link="ground"/>
-    <child link="obstacle_2"/>
-    <origin xyz="20 15 1.5" rpy="0 0 0"/>
-  </joint>
-  <link name="obstacle_3">
-    <visual>
-      <origin xyz="0 0 0" rpy="0 0 0"/>
-      <geometry>
-        <box size="4 2 5"/>
-      </geometry>
-      <material name="obstacle_color"/>
-    </visual>
-    <collision>
-      <geometry>
-        <box size="4 2 5"/>
-      </geometry>
-    </collision>
-  </link>
-  <joint name="obstacle_3_joint" type="fixed">
-    <parent link="ground"/>
-    <child link="obstacle_3"/>
-    <origin xyz="30 5 2.5" rpy="0 0 0"/>
-  </joint>
-  <link name="obstacle_4">
-    <visual>
-      <origin xyz="0 0 0" rpy="0 0 0"/>
-      <geometry>
-        <box size="2 4 2"/>
-      </geometry>
-      <material name="obstacle_color"/>
-    </visual>
-    <collision>
-      <geometry>
-        <box size="2 4 2"/>
-      </geometry>
-    </collision>
-  </link>
-  <joint name="obstacle_4_joint" type="fixed">
-    <parent link="ground"/>
-    <child link="obstacle_4"/>
-    <origin xyz="15 30 1" rpy="0 0 0"/>
-  </joint>
-  <link name="obstacle_5">
-    <visual>
-      <origin xyz="0 0 0" rpy="0 0 0"/>
-      <geometry>
-        <box size="5 1 3"/>
-      </geometry>
-      <material name="obstacle_color"/>
-    </visual>
-    <collision>
-      <geometry>
-        <box size="5 1 3"/>
-      </geometry>
-    </collision>
-  </link>
-  <joint name="obstacle_5_joint" type="fixed">
-    <parent link="ground"/>
-    <child link="obstacle_5"/>
-    <origin xyz="40 40 1.5" rpy="0 0 0"/>
-  </joint>
-  <link name="uav_start">
-    <visual>
-      <origin xyz="0 0 0" rpy="0 0 0"/>
-      <geometry>
-        <cylinder radius="0.5" length="0.01"/>
-      </geometry>
-      <material name="obstacle_color"/>
-    </visual>
-  </link>
-  <joint name="uav_start_joint" type="fixed">
-    <parent link="ground"/>
-    <child link="uav_start"/>
-    <origin xyz="0 0 0.005" rpy="0 0 0"/>
-  </joint>
-  <link name="goal">
-    <visual>
-      <origin xyz="0 0 0" rpy="0 0 0"/>
-      <geometry>
-        <cylinder radius="0.5" length="0.01"/>
-      </geometry>
-      <material name="obstacle_color"/>
-    </visual>
-  </link>
-  <joint name="goal_joint" type="fixed">
-    <parent link="ground"/>
-    <child link="goal"/>
-    <origin xyz="40 45 0.005" rpy="0 0 0"/>
-  </joint>
   <xacro:include filename="$(find fly_simulation)/urdf/quadrotor.xacro"/>
-  <xacro:quad_body_material/>
-  <xacro:quadrotor_base parent_link="uav_start">
+  <xacro:quadrotor parent_link="ground">
     <origin xyz="0 0 0.5" rpy="0 0 0"/>
-  </xacro:quadrotor_base>
+  </xacro:quadrotor>
 </robot>

File: software/fly_ROS2_sim/src/fly_simulation/urdf/quadrotor.xacro (robot description, xacro)
@@ -1,260 +1,29 @@
 <?xml version="1.0"?>
-<xml_fragment xmlns:xacro="http://www.ros.org/wiki/xacro">
-  <xacro:property name="arm_length" value="0.3"/>
-  <xacro:property name="body_width" value="0.15"/>
-  <xacro:property name="body_height" value="0.05"/>
-  <xacro:property name="propeller_radius" value="0.1"/>
-  <xacro:property name="propeller_thickness" value="0.005"/>
-  <xacro:property name="mass" value="1.5"/>
-  <xacro:macro name="quad_body_material">
-    <material name="quad_body_color">
-      <color rgba="0.3 0.3 0.3 1.0"/>
-    </material>
-    <material name="quad_arm_color">
-      <color rgba="0.5 0.5 0.5 1.0"/>
-    </material>
-    <material name="quad_propeller_color">
-      <color rgba="0.2 0.2 0.2 0.8"/>
-    </material>
+<robot xmlns:xacro="http://www.ros.org/wiki/xacro">
+  <xacro:macro name="quadrotor" params="parent_link *origin">
+    <link name="quad_base_link">
+      <visual>
+        <geometry>
+          <box size="0.3 0.3 0.1"/>
+        </geometry>
+        <material>
+          <color rgba="0.2 0.8 0.2 1"/>
+        </material>
+      </visual>
+      <collision>
+        <geometry>
+          <box size="0.3 0.3 0.1"/>
+        </geometry>
+      </collision>
+      <inertial>
+        <mass value="1.0"/>
+        <inertia ixx="0.01" ixy="0" ixz="0" iyy="0.01" iyz="0" izz="0.01"/>
+      </inertial>
+    </link>
+    <joint name="quad_base_joint" type="fixed">
+      <parent link="${parent_link}"/>
+      <child link="quad_base_link"/>
+      <xacro:insert_block name="origin"/>
+    </joint>
   </xacro:macro>
-  <xacro:macro name="quadrotor_base" params="parent_link *origin">
-  <link name="quad_base_link">
-    <visual>
-      <origin xyz="0 0 0" rpy="0 0 0"/>
-      <geometry>
-        <box size="${body_width} ${body_width} ${body_height}"/>
-      </geometry>
-      <material name="quad_body_color"/>
-    </visual>
-    <collision>
-      <origin xyz="0 0 0" rpy="0 0 0"/>
-      <geometry>
-        <box size="${body_width} ${body_width} ${body_height}"/>
-      </geometry>
-    </collision>
-    <inertial>
-      <mass value="${mass}"/>
-      <inertia ixx="0.005" ixy="0" ixz="0" iyy="0.005" iyz="0" izz="0.01"/>
-    </inertial>
-  </link>
-  <joint name="quad_base_joint" type="fixed">
-    <parent link="${parent_link}"/>
-    <child link="quad_base_link"/>
-    <xacro:insert_block name="origin"/>
-  </joint>
-  <link name="quad_front_arm">
-    <visual>
-      <origin xyz="${arm_length/2} 0 0" rpy="0 0 0"/>
-      <geometry>
-        <box size="${arm_length} 0.02 0.02"/>
-      </geometry>
-      <material name="quad_arm_color"/>
-    </visual>
-    <collision>
-      <origin xyz="${arm_length/2} 0 0" rpy="0 0 0"/>
-      <geometry>
-        <box size="${arm_length} 0.02 0.02"/>
-      </geometry>
-    </collision>
-    <inertial>
-      <mass value="0.05"/>
-      <inertia ixx="0.001" ixy="0" ixz="0" iyy="0.0001" iyz="0" izz="0.001"/>
-    </inertial>
-  </link>
-  <joint name="quad_front_arm_joint" type="fixed">
-    <parent link="quad_base_link"/>
-    <child link="quad_front_arm"/>
-    <origin xyz="0 0 0" rpy="0 0 0"/>
-  </joint>
-  <link name="quad_right_arm">
-    <visual>
-      <origin xyz="${arm_length/2} 0 0" rpy="0 0 0"/>
-      <geometry>
-        <box size="${arm_length} 0.02 0.02"/>
-      </geometry>
-      <material name="quad_arm_color"/>
-    </visual>
-    <collision>
-      <origin xyz="${arm_length/2} 0 0" rpy="0 0 0"/>
-      <geometry>
-        <box size="${arm_length} 0.02 0.02"/>
-      </geometry>
-    </collision>
-    <inertial>
-      <mass value="0.05"/>
-      <inertia ixx="0.001" ixy="0" ixz="0" iyy="0.0001" iyz="0" izz="0.001"/>
-    </inertial>
-  </link>
-  <joint name="quad_right_arm_joint" type="fixed">
-    <parent link="quad_base_link"/>
-    <child link="quad_right_arm"/>
-    <origin xyz="0 0 0" rpy="0 0 1.5708"/>
-  </joint>
-  <link name="quad_back_arm">
-    <visual>
-      <origin xyz="${arm_length/2} 0 0" rpy="0 0 0"/>
-      <geometry>
-        <box size="${arm_length} 0.02 0.02"/>
-      </geometry>
-      <material name="quad_arm_color"/>
-    </visual>
-    <collision>
-      <origin xyz="${arm_length/2} 0 0" rpy="0 0 0"/>
-      <geometry>
-        <box size="${arm_length} 0.02 0.02"/>
-      </geometry>
-    </collision>
-    <inertial>
-      <mass value="0.05"/>
-      <inertia ixx="0.001" ixy="0" ixz="0" iyy="0.0001" iyz="0" izz="0.001"/>
-    </inertial>
-  </link>
-  <joint name="quad_back_arm_joint" type="fixed">
-    <parent link="quad_base_link"/>
-    <child link="quad_back_arm"/>
-    <origin xyz="0 0 0" rpy="0 0 3.14159"/>
-  </joint>
-  <link name="quad_left_arm">
-    <visual>
-      <origin xyz="${arm_length/2} 0 0" rpy="0 0 0"/>
-      <geometry>
-        <box size="${arm_length} 0.02 0.02"/>
-      </geometry>
-      <material name="quad_arm_color"/>
-    </visual>
-    <collision>
-      <origin xyz="${arm_length/2} 0 0" rpy="0 0 0"/>
-      <geometry>
-        <box size="${arm_length} 0.02 0.02"/>
-      </geometry>
-    </collision>
-    <inertial>
-      <mass value="0.05"/>
-      <inertia ixx="0.001" ixy="0" ixz="0" iyy="0.0001" iyz="0" izz="0.001"/>
-    </inertial>
-  </link>
-  <joint name="quad_left_arm_joint" type="fixed">
-    <parent link="quad_base_link"/>
-    <child link="quad_left_arm"/>
-    <origin xyz="0 0 0" rpy="0 0 -1.5708"/>
-  </joint>
-  <link name="quad_front_prop">
-    <visual>
-      <origin xyz="0 0 0" rpy="0 0 0"/>
-      <geometry>
-        <cylinder radius="${propeller_radius}" length="${propeller_thickness}"/>
-      </geometry>
-      <material name="quad_propeller_color"/>
-    </visual>
-    <collision>
-      <origin xyz="0 0 0" rpy="0 0 0"/>
-      <geometry>
-        <cylinder radius="${propeller_radius}" length="${propeller_thickness}"/>
-      </geometry>
-    </collision>
-    <inertial>
-      <mass value="0.01"/>
-      <inertia ixx="0.0001" ixy="0" ixz="0" iyy="0.0001" iyz="0" izz="0.0001"/>
-    </inertial>
-  </link>
-  <joint name="quad_front_prop_joint" type="continuous">
-    <parent link="quad_front_arm"/>
-    <child link="quad_front_prop"/>
-    <origin xyz="${arm_length} 0 0" rpy="0 0 0"/>
-    <axis xyz="0 0 1"/>
-  </joint>
-  <link name="quad_right_prop">
-    <visual>
-      <origin xyz="0 0 0" rpy="0 0 0"/>
-      <geometry>
-        <cylinder radius="${propeller_radius}" length="${propeller_thickness}"/>
-      </geometry>
-      <material name="quad_propeller_color"/>
-    </visual>
-    <collision>
-      <origin xyz="0 0 0" rpy="0 0 0"/>
-      <geometry>
-        <cylinder radius="${propeller_radius}" length="${propeller_thickness}"/>
-      </geometry>
-    </collision>
-    <inertial>
-      <mass value="0.01"/>
-      <inertia ixx="0.0001" ixy="0" ixz="0" iyy="0.0001" iyz="0" izz="0.0001"/>
-    </inertial>
-  </link>
-  <joint name="quad_right_prop_joint" type="continuous">
-    <parent link="quad_right_arm"/>
-    <child link="quad_right_prop"/>
-    <origin xyz="${arm_length} 0 0" rpy="0 0 0"/>
-    <axis xyz="0 0 1"/>
-  </joint>
-  <link name="quad_back_prop">
-    <visual>
-      <origin xyz="0 0 0" rpy="0 0 0"/>
-      <geometry>
-        <cylinder radius="${propeller_radius}" length="${propeller_thickness}"/>
-      </geometry>
-      <material name="quad_propeller_color"/>
-    </visual>
-    <collision>
-      <origin xyz="0 0 0" rpy="0 0 0"/>
-      <geometry>
-        <cylinder radius="${propeller_radius}" length="${propeller_thickness}"/>
-      </geometry>
-    </collision>
-    <inertial>
-      <mass value="0.01"/>
-      <inertia ixx="0.0001" ixy="0" ixz="0" iyy="0.0001" iyz="0" izz="0.0001"/>
-    </inertial>
-  </link>
-  <joint name="quad_back_prop_joint" type="continuous">
-    <parent link="quad_back_arm"/>
-    <child link="quad_back_prop"/>
-    <origin xyz="${arm_length} 0 0" rpy="0 0 0"/>
-    <axis xyz="0 0 1"/>
-  </joint>
-  <link name="quad_left_prop">
-    <visual>
-      <origin xyz="0 0 0" rpy="0 0 0"/>
-      <geometry>
-        <cylinder radius="${propeller_radius}" length="${propeller_thickness}"/>
-      </geometry>
-      <material name="quad_propeller_color"/>
-    </visual>
-    <collision>
-      <origin xyz="0 0 0" rpy="0 0 0"/>
-      <geometry>
-        <cylinder radius="${propeller_radius}" length="${propeller_thickness}"/>
-      </geometry>
-    </collision>
-    <inertial>
-      <mass value="0.01"/>
-      <inertia ixx="0.0001" ixy="0" ixz="0" iyy="0.0001" iyz="0" izz="0.0001"/>
-    </inertial>
-  </link>
-  <joint name="quad_left_prop_joint" type="continuous">
-    <parent link="quad_left_arm"/>
-    <child link="quad_left_prop"/>
-    <origin xyz="${arm_length} 0 0" rpy="0 0 0"/>
-    <axis xyz="0 0 1"/>
-  </joint>
-  <link name="quad_imu_link">
-    <visual>
-      <origin xyz="0 0 0" rpy="0 0 0"/>
-      <geometry>
-        <box size="0.03 0.03 0.02"/>
-      </geometry>
-      <material name="quad_body_color"/>
-    </visual>
-    <inertial>
-      <mass value="0.01"/>
-      <inertia ixx="0.00001" ixy="0" ixz="0" iyy="0.00001" iyz="0" izz="0.00001"/>
-    </inertial>
-  </link>
-  <joint name="quad_imu_joint" type="fixed">
-    <parent link="quad_base_link"/>
-    <child link="quad_imu_link"/>
-    <origin xyz="0 0 -0.02" rpy="0 0 0"/>
-  </joint>
-  </xacro:macro>
-</xml_fragment>
+</robot>
